File: Nodo 2 MySensor Kicad/Nodo 2 MySensor.kicad_sch (KiCad schematic)
At the start: 9 parts, among them J1 FTDI, J2 I2C, J3 Analog, J4 Conn_01x06_Pin, J5 Conn_01x06_Pin, J6 Analog, J7 Digital, J8 2060-452_998-404, U1 NRF24L01_Breakout

Commit message: Diseño del nodo 2 placa
Parts:
- J8: footprint 2060-452_998-404:WAGO_2060-452_998-404 -> ee:WAGO_2060-452_998-404
Changed lines of the file:
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@@
 			)
 		)
-		(property "Footprint" "2060-452_998-404:WAGO_2060-452_998-404"
+		(property "Footprint" "ee:WAGO_2060-452_998-404"
 			(at 33.02 96.52 0)
 			(effects
