File: Nodo 2 MySensor Kicad/Nodo 2 MySensor.kicad_pcb (KiCad board)
At the start: 2 copper layers, 33 x 17.8 mm, 5 parts, among them J1 FTDI, J2 I2C, J3 Analog, J6 Analog, J7 Digital

Commit message: Diseño del nodo 2 placa
Parts:
- removed J3: Analog, Connector_PinHeader_2.54mm:PinHeader_1x02_P2.54mm_Vertical
- added ?: , , F.Cu at (131.8, 91.1)
- added ?: , , F.Cu at (131.8, 88.6)
- added ?: , , F.Cu at (131.8, 86.0)
- added J4: Conn_01x06_Pin, Connector_PinHeader_2.54mm:PinHeader_1x06_P2.54mm_Vertical_SMD_Pin1Right, F.Cu at (81.4, 90.9)
- added J5: Conn_01x06_Pin, Connector_PinHeader_2.54mm:PinHeader_1x06_P2.54mm_Vertical_SMD_Pin1Right, F.Cu at (145.4, 91.9)
- added J8: 2060-452_998-404, ee:WAGO_2060-452_998-404, F.Cu at (88.0, 67.3)
- added U1: NRF24L01_Breakout, Connector_PinHeader_2.54mm:PinHeader_2x04_P2.54mm_Vertical_SMD, F.Cu at (126.8, 66.9)
Connections:
- J1 pad 1: GND -> /DTR
- J1 pad 2: GND -> /TX
- J1 pad 3: VCC -> /RX
- J1 pad 4: /RX -> VCC
- J1 pad 5: /TX -> GND
- J1 pad 6: /DTR -> GND
Routing:
- net VCC: track 0.00 -> 134.6 mm
- net GND: track 0.00 -> 120.8 mm
- net /*D9: track 0.00 -> 95.0 mm
- net /SS/*D10: track 0.00 -> 39.4 mm
- net /SDA/A4: track 0.00 -> 35.7 mm
- net /SCL/A5: track 0.00 -> 34.5 mm
- net /MOSI/*D11: track 0.00 -> 24.6 mm
- net /RX: track 0.00 -> 22.1 mm
- net /DTR: track 0.00 -> 22.1 mm
- net /TX: track 0.00 -> 18.8 mm
- net /SCK/D13: track 0.00 -> 15.7 mm
- net /MISO/D12: track 0.00 -> 15.7 mm
Other:
- board outline removed
- board text added: "A.J.G.R. & C.J.B."

Commit message: Nodo 1 esquematico
Parts:
- removed ? (x3): , 
- moved J8 9.75 mm to (95.8, 73.1), turned to -90 degrees
- moved J4 5.40 mm to (86.8, 90.7)
- moved U1 4.91 mm to (127.6, 71.7)
- moved J5 3.50 mm to (142.0, 91.0)
Routing:
- net /*D9: track 95.0 -> 76.3 mm
- net GND: track 120.8 -> 104.3 mm
- net /SS/*D10: track 39.4 -> 31.5 mm
- net VCC: track 134.6 -> 126.6 mm
- net /DTR: track 22.1 -> 16.4 mm
- net /MOSI/*D11: track 24.6 -> 19.1 mm
- net /SCK/D13: track 15.7 -> 11.2 mm
- net /MISO/D12: track 15.7 -> 11.2 mm
- net /RX: track 22.1 -> 26.3 mm
- net /SDA/A4: track 35.7 -> 32.6 mm
- net /SCL/A5: track 34.5 -> 33.5 mm
Other:
- board text added: "${REFERENCE}"
