File: Nodo 1 MySensor Kicad/Nodo 1 MySensor Kicad.kicad_pcb (KiCad board)
At the start: 2 copper layers, 22 parts, among them J2 I2C, J4 Conn_01x06, J6 Analog, J7 Digital, K1 OJE-SS-112LMH_000, Q1 BC547, U1 NRF24L01_Breakout

Commit message: Conexion del nodo 1
Parts:
- removed the ? at (78.5, 123.1)
- removed the ? at (78.5, 120.5)
- removed the ? at (78.5, 118.0)
- removed R1: R, Resistor_SMD:R_1206_3216Metric_Pad1.30x1.75mm_HandSolder
- added F1: Fuse, Fuse:Fuseholder_Cylinder-5x20mm_Schurter_0031_8201_Horizontal_Open, F.Cu at (267.2, 74.5)
- added F2: Fuse, Resistor_THT:R_Axial_DIN0414_L11.9mm_D4.5mm_P15.24mm_Horizontal, F.Cu at (234.7, 89.5)
- added F3: Fuse, Fuse:Fuseholder_Cylinder-5x20mm_Schurter_0031_8201_Horizontal_Open, F.Cu at (225.9, 95.0)
- added J2: I2C, Connector_PinHeader_2.54mm:PinHeader_1x02_P2.54mm_Vertical, F.Cu at (251.1, 55.1)
- added J4: Conn_01x06, TerminalBlock:TerminalBlock_bornier-6_P5.08mm, F.Cu at (225.0, 67.6)
- added J6: Analog, Connector_PinHeader_2.54mm:PinHeader_1x12_P2.54mm_Vertical, B.Cu at (239.7, 52.2)
- added J7: Digital, Connector_PinHeader_2.54mm:PinHeader_1x12_P2.54mm_Vertical, B.Cu at (267.6, 67.4)
- added K1: OJE-SS-112LMH_000, OJE-SS-112LMH_000.:TE_5-1419128-0, F.Cu at (260.3, 85.4)
- added PS1: HLK-PM01, Converter_ACDC:Converter_ACDC_Hi-Link_HLK-PMxx, F.Cu at (236.0, 100.5)
- added Q1: BC547, Package_TO_SOT_THT:TO-92_Inline, F.Cu at (243.4, 46.3)
- added RV1: Varistor, Varistor:RV_Disc_D12mm_W6.2mm_P7.5mm, F.Cu at (248.2, 89.3)
- added U1: NRF24L01_Breakout, RF_Module:nRF24L01_Breakout, F.Cu at (260.0, 48.2)
- moved Q1 2.99 mm to (53.7, 109.4), turned to -90 degrees
Routing:
- net Net-(Q1-C): track 0.00 -> 156.6 mm
- net VCC: track 0.00 -> 61.6 mm
- net /AC+: track 27.7 -> 76.2 mm
- net GND: track 0.00 -> 48.4 mm
- net /D7: track 0.00 -> 41.7 mm
- net /*D6: track 0.00 -> 37.0 mm
- net /*D9: track 0.00 -> 24.8 mm
- net /SS/*D10: track 0.00 -> 16.1 mm
- net /MOSI/*D11: track 0.00 -> 13.1 mm
- net /SCK/D13: track 0.00 -> 6.59 mm
- net /MISO/D12: track 0.00 -> 6.15 mm
